File: pcb/lightrail_dual_nce.kicad_pcb (KiCad board)
At the start: 32 copper layers, 420 x 350 mm, 0 parts

Commit message: Pour the plane layers; make the fab export reproducible and self-verifying
build_board.py named 15 layers GND1..GND29 and VDD3..VDD27 but the board held
zero zones, so all 15 were empty copper. The export looked right -- 32 copper
Gerbers with the correct names -- and would have shipped as bare laminate on
15 layers. add_planes.py pours them; the planes now carry copper on the GND
and VDD nets.

Three supporting changes.

export_fab.sh replaces the hand-typed kicad-cli calls that produced the first
package. Those were not reproducible and went stale the moment the copper
changed, which is exactly what just happened. Two flag errors found writing
it: --no-protel-ext is a boolean opt-out and takes no value, and drill units
are --excellon-units, not --units. Both failed silently under set -e by
printing usage.

verify_fab.py parses the exported Gerbers rather than trusting the plot
result, and the export now gates on it. It initially reported 0 plane layers
on a package that was in fact correct: KiCad 10 emits no %LayerName attribute
on copper, so the detector found nothing. It now keys on %TO.N, which is the
stronger check -- it confirms the pour landed on the right rail, which a layer
name cannot tell you.

Measured for the PDN: 1 oz sheet resistance 0.4914 mohm/square, 7 VDD planes
in parallel give 14.6 uohm against the 24 uohm target. Stated carefully, this
does not contradict l01_pdn.py's 296x shortfall -- plane spreading is the most
favourable term in the budget and this excludes via, package, ball and on-die
resistance. The only conclusion it supports is that the deficit is not in the
planes, so adding plane layers will not close it.

DRC moved from 0 violations to 15, all warnings, all isolated_copper, one per
plane. Not suppressed: a plane whose net has no pads really is isolated, and
the warning is DRC reporting the missing schematic. It could not report it
before because there was no copper to be isolated. Errors stay at 0 and the
export gates on errors only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
Routing:
- added copper zone on In1.Cu, net GND
- added copper zone on In13.Cu, net GND
- added copper zone on In17.Cu, net GND
- added copper zone on In21.Cu, net GND
- added copper zone on In25.Cu, net GND
- added copper zone on In29.Cu, net GND
- added copper zone on In5.Cu, net GND
- added copper zone on In9.Cu, net GND
- added copper zone on In11.Cu, net VDD
- added copper zone on In15.Cu, net VDD
- added copper zone on In19.Cu, net VDD
- added copper zone on In23.Cu, net VDD
- added copper zone on In27.Cu, net VDD
- added copper zone on In3.Cu, net VDD
- added copper zone on In7.Cu, net VDD

Commit message: Repair build_board.py, which could not run, and make the board pipeline work
build_board.py has been syntactically broken on disk: line 177 held
newline="<actual newline>" instead of the escape, so the module raised
SyntaxError on import and the script could not execute at all. Nothing
caught it because nothing had re-run it since the corruption; the project
file it writes was left over from an earlier run.

The consequence was not confined to that file. add_planes.py was not
idempotent, so when build_board.py silently failed to regenerate the board,
add_planes added a second zone to all 15 plane layers -- 30 overlapping
fills on a board that should have had 15. It now clears existing zones
first.

build_all.sh runs the three stages in dependency order and reports real
failures. Its first version ended each pipeline with "|| true" and then read
PIPESTATUS, which described the "|| true" rather than the Python process, so
it reported success while build_board.py was dying. Same class of mistake as
piping a build into head, which earlier sent SIGPIPE to build_schematic.py
and masked a crash as exit 0; both are now avoided by capturing status
before filtering output.

Three KiCad 10 binding defects worked around, each found by hitting it:
  - GetDrawings() calls list() on a non-iterable SwigPyObject
  - Drawings() advertises __iter__ but raises TypeError when iterated, and
    loses len() once footprints have been removed
  - PAD positions cannot be set relative to a parent, because
    FOOTPRINT.GetPosition() returns an object with no .x
Rather than keep probing the drawings API, build_board.py now takes
--no-markers and never draws the placeholder silkscreen. Not creating
artwork beats deleting it.

Pipeline now completes: 32 copper layers, 15 plane zones, 51 components,
5368 pads, 931 nets, 48 DrMOS phases.

Co-Authored-By: Claude Opus 5 <noreply@anthropic.com>
Parts:
- added PIC1: TFLN-BRIDGE-3T2, , F.Cu at (210.0, 175.0)
- added U1: NCE-BGA2500, , F.Cu at (152.5, 175.0)
- added U100: DrMOS, , F.Cu at (50.0, 20.0)
- added U101: DrMOS, , F.Cu at (79.1, 20.0)
- added U102: DrMOS, , F.Cu at (108.2, 20.0)
- added U103: DrMOS, , F.Cu at (137.3, 20.0)
- added U104: DrMOS, , F.Cu at (166.4, 20.0)
- added U105: DrMOS, , F.Cu at (195.5, 20.0)
- added U106: DrMOS, , F.Cu at (224.5, 20.0)
- added U107: DrMOS, , F.Cu at (253.6, 20.0)
- added U108: DrMOS, , F.Cu at (282.7, 20.0)
- added U109: DrMOS, , F.Cu at (311.8, 20.0)
- added U110: DrMOS, , F.Cu at (340.9, 20.0)
- added U111: DrMOS, , F.Cu at (370.0, 20.0)
- added U112: DrMOS, , F.Cu at (50.0, 28.0)
- added U113: DrMOS, , F.Cu at (79.1, 28.0)
- added U114: DrMOS, , F.Cu at (108.2, 28.0)
- added U115: DrMOS, , F.Cu at (137.3, 28.0)
- added U116: DrMOS, , F.Cu at (166.4, 28.0)
- added U117: DrMOS, , F.Cu at (195.5, 28.0)
- added U118: DrMOS, , F.Cu at (224.5, 28.0)
- added U119: DrMOS, , F.Cu at (253.6, 28.0)
- added U120: DrMOS, , F.Cu at (282.7, 28.0)
- added U121: DrMOS, , F.Cu at (311.8, 28.0)
- added U122: DrMOS, , F.Cu at (340.9, 28.0)
- added U123: DrMOS, , F.Cu at (370.0, 28.0)
- added U124: DrMOS, , F.Cu at (50.0, 324.0)
- added U125: DrMOS, , F.Cu at (79.1, 324.0)
- added U126: DrMOS, , F.Cu at (108.2, 324.0)
- added U127: DrMOS, , F.Cu at (137.3, 324.0)
- added U128: DrMOS, , F.Cu at (166.4, 324.0)
- added U129: DrMOS, , F.Cu at (195.5, 324.0)
- added U130: DrMOS, , F.Cu at (224.5, 324.0)
- added U131: DrMOS, , F.Cu at (253.6, 324.0)
- added U132: DrMOS, , F.Cu at (282.7, 324.0)
- added U133: DrMOS, , F.Cu at (311.8, 324.0)
- added U134: DrMOS, , F.Cu at (340.9, 324.0)
- added U135: DrMOS, , F.Cu at (370.0, 324.0)
- added U136: DrMOS, , F.Cu at (50.0, 316.0)
- added U137: DrMOS, , F.Cu at (79.1, 316.0)
- added U138: DrMOS, , F.Cu at (108.2, 316.0)
- added U139: DrMOS, , F.Cu at (137.3, 316.0)
- added U140: DrMOS, , F.Cu at (166.4, 316.0)
- added U141: DrMOS, , F.Cu at (195.5, 316.0)
- added U142: DrMOS, , F.Cu at (224.5, 316.0)
- added U143: DrMOS, , F.Cu at (253.6, 316.0)
- added U144: DrMOS, , F.Cu at (282.7, 316.0)
- added U145: DrMOS, , F.Cu at (311.8, 316.0)
- added U146: DrMOS, , F.Cu at (340.9, 316.0)
- added U147: DrMOS, , F.Cu at (370.0, 316.0)
- added U2: NCE-BGA2500, , F.Cu at (267.5, 175.0)
Other:
- board text removed: "NCE DIE A"
- board text removed: "NCE DIE B"
- board text removed: "TFLN PIC"
- board text removed: "U000"
- board text removed: "U001"
- board text removed: "U002"
- board text removed: "U003"
- board text removed: "U004"
- board text removed: "U005"
- board text removed: "U006"
- board text removed: "U007"
- board text removed: "U008"
- board text removed: "U009"
- board text removed: "U010"
- board text removed: "U011"
- board text removed: "U100"
- board text removed: "U101"
- board text removed: "U102"
- board text removed: "U103"
- board text removed: "U104"
- board text removed: "U105"
- board text removed: "U106"
- board text removed: "U107"
- board text removed: "U108"
- board text removed: "U109"
- board text removed: "U110"
- board text removed: "U111"
