File: pcb/lightrail_dual_nce.kicad_pcb (KiCad board)
At the start: 32 copper layers, 420 x 350 mm, 51 parts, among them U1 NCE-BGA2500, U100 DrMOS, U101 DrMOS, U102 DrMOS, U103 DrMOS, U104 DrMOS, U105 DrMOS, U106 DrMOS, U107 DrMOS, U108 DrMOS, U109 DrMOS, U110 DrMOS, U111 DrMOS, U112 DrMOS, U113 DrMOS, U114 DrMOS, U115 DrMOS, U116 DrMOS, U117 DrMOS, U118 DrMOS, U119 DrMOS, U120 DrMOS, U121 DrMOS, U122 DrMOS, U123 DrMOS, U124 DrMOS, U125 DrMOS, U126 DrMOS, U127 DrMOS, U128 DrMOS, U129 DrMOS, U130 DrMOS, U131 DrMOS, U132 DrMOS, U133 DrMOS, U134 DrMOS, U135 DrMOS, U136 DrMOS, U137 DrMOS, U138 DrMOS, U139 DrMOS, U140 DrMOS, U141 DrMOS, U142 DrMOS, U143 DrMOS, U144 DrMOS, U145 DrMOS, U146 DrMOS, U147 DrMOS, U2 NCE-BGA2500

Commit message: Add custom DRC rules, optical keep-out, HBM4 placement and a master harness
Four items from the agreed plan. Three findings came out of building them.

The 12:1 aspect-ratio cap is incompatible with the current drill. KiCad has
no board-thickness variable, so a ratio has to be converted to a minimum
hole size at the known thickness, and that conversion is the result: at the
4.54 mm stackup, 12:1 needs a drill of at least 0.378 mm. The project rule
is 0.30 mm, which is 15.1:1 and fails the cap. nce_custom_rules.kicad_dru
sets 0.40 mm, giving 11.35:1, and the project file has to move with it.

The rule was described as a MICROVIA constraint. It is not. A microvia
spans one 0.110 mm dielectric gap rather than the board, so at a 0.10 mm
drill it is 1.10:1 -- nowhere near 12:1. What limits a microvia is laser
drilling and plating. The 12:1 figure is a through-via rule and is written
as one.

The optical corridor as specified cannot be enforced. X = [110..310] mm
contains U1 (125..180), U2 (240..295) and PIC1 (185..235) in their
entirety, so a copper-free zone there forbids all 5400 pads and both dies.
The corridor matching the intent is the 60 mm optical gap, X = [180..240],
which is where the PIC already sits. It is built as specified so DRC can
show the consequence rather than have it argued.

HBM4 stacks go above and below each die rather than beside it: the inner
faces are where the optical lanes escape toward the PIC and the outer faces
carry the power feed. Four pads each, not 1024 -- this is a placement
study, and putting 8192 undriven pads on the board would misrepresent it.

run_master_verification.py wraps the existing suites and reports their real
exit codes. It reimplements no check, because a harness that prints its own
version of a result is a second source of truth and the second one drifts.
A suite needing the EDA container reports UNAVAILABLE and FAILS the run
rather than letting the reachable subset pass.

Verified in hpretl/iic-osic-tools: 7 of 7 suite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
Parts:
- added MA00: HBM4-12Hi, , F.Cu at (145.5, 139.0)
- added MA01: HBM4-12Hi, , F.Cu at (159.5, 139.0)
- added MA10: HBM4-12Hi, , F.Cu at (145.5, 211.0)
- added MA11: HBM4-12Hi, , F.Cu at (159.5, 211.0)
- added MB00: HBM4-12Hi, , F.Cu at (260.5, 139.0)
- added MB01: HBM4-12Hi, , F.Cu at (274.5, 139.0)
- added MB10: HBM4-12Hi, , F.Cu at (260.5, 211.0)
- added MB11: HBM4-12Hi, , F.Cu at (274.5, 211.0)
